File: Sundial_min/Sundial_min.kicad_sch (KiCad schematic)
At the start: 90 parts, among them SW1 RotaryEncoder_Switch, SW2 RotaryEncoder_Switch, SW3 RotaryEncoder_Switch

Commit message: battery manager work
Parts:
- added C1, C2, C3: 10u, symbol Device:C
- added C4, C5: 4u7, symbol Device:C
- added D27, D32: LED, symbol Device:LED
- added J1: USB_C_Receptacle_USB2.0_16P, symbol Connector:USB_C_Receptacle_USB2.0_16P
- added J2: Conn_01x02, symbol Connector_Generic:Conn_01x02
- added R1, R2: 5.1k, symbol Device:R
- added R3: 10k, symbol Device:R
- added R4: 10K, symbol Device:R
- added R6, R7: 1k, symbol Device:R
- added SW4: SW_Push, symbol Switch:SW_Push
- added U1: E73-2G4M08S1C, E73-2G4M08S1C:E73-2G4M08S1C, symbol E73-2G4M08S1C:E73-2G4M08S1C
- added U2: BQ24075RGT, Package_DFN_QFN:VQFN-16-1EP_3x3mm_P0.5mm_EP1.6x1.6mm, symbol Battery_Management:BQ24075RGT
- added U3: NCP1117-3.3_SOT223, Package_TO_SOT_SMD:SOT-223-3_TabPin2, symbol Regulator_Linear:NCP1117-3.3_SOT223
Connections:
- net GND: now also C1.2, C2.2, C3.1, C4.2, C5.2, J1.A1 (GND), J1.A12 (GND), J1.B1 (GND), J1.B12 (GND), J1.SH (SHIELD), J2.2 (Pin_2), R1.1, R2.2, R3.2, SW4.2, U1.21 (GND@2), U1.24 (GND@3), U1.5 (GND@1), U2.4 (~{CE}), U3.1 (GND)
- new net: J1.B5 (CC2), R2.1
- new net: R3.1, U2.1 (TS)
- new net: U2.17 (VSS), U2.8 (VSS)
- new net: D27.1 (K), U2.7 (~{PGOOD})
- new net: D32.1 (K), U2.9 (~{CHG})
- new net: D27.2 (A), R6.1
- new net: J1.A5 (CC1), R1.2
- new net: D32.2 (A), R7.1
- new net +3V3: C2.1, C3.2, R4.2, U1.19 (VDD), U1.23 (VDDH), U3.2 (VO)
- new net +5V: J1.A4 (VBUS), J1.A9 (VBUS), J1.B4 (VBUS), J1.B9 (VBUS), U1.27 (VBUS), U2.13 (IN)
- new net BAT: C5.1, J2.1 (Pin_1), U2.2 (BAT), U2.3 (BAT)
- new net D+: J1.A6 (D+), J1.B6 (D+), U1.31 (DP)
- new net D-: J1.A7 (D-), J1.B7 (D-), U1.29 (DM)
- new net SWDCLK: U1.39 (SWDCLK)
- new net SWDIO: U1.37 (SWDIO)
- new net VCC: C1.1, C4.1, R6.2, R7.2, U2.10 (OUT), U2.11 (OUT), U2.5 (EN2), U3.3 (VI)
- new net ~{RESET}: R4.1, SW4.1, U1.26 (P0.18/RESET)
- no-connect marks 0 -> 3
Other:
- note added: "Battery Manager"
- note added: "LDO"
- moved on the sheet: D1, D10, D11, D12, D13, D14, D15, D16, D17, D18, D19, D2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

Commit message: battery manager
Parts:
- added R2: 47K, symbol Device:R
- added R3: 1.5K, symbol Device:R
- added R4: 3K, symbol Device:R
- added SW5: SW_Push, symbol Switch:SW_Push
- J1: renamed from J2; value Conn_01x02 -> Battery Connecter
- renumbered C3 to C1, C5 to C2, C1 to C3, C2 to C4, C4 to C5, D25 to D1, D13 to D10, D14 to D11, D3 to D12, D8 to D13, D15 to D14, D16 to D15, D4 to D16, D9 to D17, D17 to D18, D18 to D19, D23 to D2, D5 to D20, D10 to D21, D19 to D22, D20 to D23, D21 to D24, D22 to D25, D28 to D26, D29 to D27, D30 to D28, D31 to D29, D24 to D3, D33 to D30, D34 to D31, D35 to D32, D36 to D33, D38 to D34, D39 to D35, D40 to D36, D41 to D37, D43 to D38, D44 to D39, D1 to D4, D45 to D40, D46 to D41, D48 to D42, D49 to D43, D50 to D44, D51 to D45, D27 to D46, D32 to D47, D6 to D5, D11 to D6, D12 to D7, D2 to D8, D7 to D9, J1 to J2, R4 to R1, R3 to R5, R1 to R8, R2 to R9, S8 to S10, S15 to S11, S16 to S12, S4 to S13, S9 to S14, S17 to S15, S18 to S16, S5 to S17, S10 to S18, S6 to S2, S28 to S23, S29 to S24, S30 to S25, S31 to S26, S33 to S27, S34 to S28, S35 to S29, S11 to S3, S36 to S30, S38 to S31, S39 to S32, S40 to S33, S41 to S34, S43 to S35, S44 to S36, S45 to S37, S46 to S38, S48 to S39, S12 to S4, S49 to S40, S50 to S41, S51 to S42, S2 to S5, S7 to S6, S13 to S7, S14 to S8, S3 to S9
Connections:
- net GND: now also U2.17 (VSS), U2.6 (EN1), U2.8 (VSS), R2.1, R3.1, R4.1, SW5.1
- net at U2.12 (ILIM): now also R3.2
- net at U2.14 (TMR): now also R2.2
- net at U2.15 (SYSOFF): now also SW5.2
- net at U2.16 (ISET): now also R4.2
Other:
- moved on the sheet: C2, D1, D2, D3, J1
